Commit message: bug fix

File: src/husky_ws/src/husky/husky_description/urdf/husky.urdf.xacro (robot description, xacro)
@@ -39,4 +39,5 @@
   <xacro:include filename="$(find husky_description)/urdf/accessories/sick_lms1xx_mount.urdf.xacro"/>
   <xacro:include filename="$(find husky_description)/urdf/accessories/sensor_arch.urdf.xacro"/>
+   <!-- <xacro:include filename="$(find gazebo_ros_battery)/xacro/battery.xacro"/> -->
   <xacro:property name="M_PI" value="3.14159"/>
   <!-- Base Size -->
@@ -146,4 +147,28 @@
     <xacro:intel_realsense_mount prefix="camera" topic="realsense" parent_link="realsense_mountpoint"/>
   </xacro:if>
+  <!-- battery -->
+  <!-- <link name="battery_link"/>
+  <joint name="battery_joint" type="fixed">
+    <parent link="base_link"/>
+    <child link="battery_link"/>
+  </joint>
+  <xacro:battery sensor_name="battery" frame_id="battery_link"
+                 params_yaml="$(find gazebo_ros_battery)/params/G24B4.yaml"/> -->
+<!-- bumper -->
+  <!-- <gazebo reference="base_link">
+    <sensor name="bumper_sensor" type="contact">
+        <selfCollide>true</selfCollide>
+        <alwaysOn>true</alwaysOn>
+        <updateRate>15.0</updateRate>
+        <material>Gazebo/Red</material>
+        <contact>
+            <collision>base_link_collision</collision>
+        </contact>
+        <plugin name="gazebo_ros_bumper_controller" filename="libgazebo_ros_bumper.so">
+            <bumperTopicName>bumper_vals</bumperTopicName>
+            <frameName>world</frameName>
+        </plugin>
+    </sensor>
+</gazebo> -->
 <!-- <gazebo>
   <plugin name="ros_bumper_controller" filename="libgazebo_ros_bumper.so">

Commit message: added battery and collision detection

File: src/husky_ws/src/husky/husky_description/urdf/husky.urdf.xacro (robot description, xacro)
@@ -39,5 +39,5 @@
   <xacro:include filename="$(find husky_description)/urdf/accessories/sick_lms1xx_mount.urdf.xacro"/>
   <xacro:include filename="$(find husky_description)/urdf/accessories/sensor_arch.urdf.xacro"/>
-   <!-- <xacro:include filename="$(find gazebo_ros_battery)/xacro/battery.xacro"/> -->
+   <xacro:include filename="$(find gazebo_ros_battery)/xacro/battery.xacro"/>
   <xacro:property name="M_PI" value="3.14159"/>
   <!-- Base Size -->
@@ -148,5 +148,5 @@
   </xacro:if>
   <!-- battery -->
-  <!-- <link name="battery_link"/>
+  <link name="battery_link"/>
   <joint name="battery_joint" type="fixed">
     <parent link="base_link"/>
@@ -154,11 +154,11 @@
   </joint>
   <xacro:battery sensor_name="battery" frame_id="battery_link"
-                 params_yaml="$(find gazebo_ros_battery)/params/G24B4.yaml"/> -->
+                 params_yaml="$(find gazebo_ros_battery)/params/my_custom_config.yaml"/>
 <!-- bumper -->
-  <!-- <gazebo reference="base_link">
+  <gazebo reference="base_link">
     <sensor name="bumper_sensor" type="contact">
         <selfCollide>true</selfCollide>
         <alwaysOn>true</alwaysOn>
-        <updateRate>15.0</updateRate>
+        <updateRate>1.0</updateRate>
         <material>Gazebo/Red</material>
         <contact>
@@ -170,14 +170,5 @@
         </plugin>
     </sensor>
-</gazebo> -->
-<!-- <gazebo>
-  <plugin name="ros_bumper_controller" filename="libgazebo_ros_bumper.so">
-    <robotNamespace>$(arg robot_namespace)</robotNamespace>
-    <alwaysOn>true</alwaysOn>
-    <updateRate>50</updateRate>
-    <bumperTopicName>husky/collision</bumperTopicName>
-    <frameName>world</frameName>
-  </plugin>
-</gazebo>   -->
+</gazebo>
   <gazebo>
     <plugin name="gazebo_ros_control" filename="libgazebo_ros_control.so">
